File: pcb/galvanize/galvanize.sch (KiCad schematic (older format))
At the start: 23 parts

Commit message: Add pcb files to repo.
Parts:
- removed J? (x2): Conn_01x14, symbol Connector_Generic:Conn_01x14
- added C1, C2, C3: C, Capacitor_SMD:C_0805_2012Metric_Pad1.15x1.40mm_HandSolder, symbol Device:C
- J1: renamed from J?; value Conn_01x02 -> RIGHT; footprint (none) -> galvanize:PinHeader_1x02_P2.54mm_Vertical_Labeled
- J10: renamed from J?; value Conn_01x02 -> B6; footprint (none) -> galvanize:PinHeader_1x02_P2.54mm_Vertical_Labeled
- J11: renamed from J?; value Conn_01x02 -> B7; footprint (none) -> galvanize:PinHeader_1x02_P2.54mm_Vertical_Labeled
- J12: renamed from J?; value Conn_01x02 -> B8; footprint (none) -> galvanize:PinHeader_1x02_P2.54mm_Vertical_Labeled
- J13: renamed from J?; value Conn_01x02 -> B9; footprint (none) -> galvanize:PinHeader_1x02_P2.54mm_Vertical_Labeled
- J14: renamed from J?; value Conn_01x02 -> 10; footprint (none) -> galvanize:PinHeader_1x02_P2.54mm_Vertical_Labeled
- J15: renamed from J?; value Conn_01x03 -> L_X; footprint (none) -> galvanize:PinHeader_1x03_P2.54mm_Vertical_Labeled
- J16: renamed from J?; value Conn_01x03 -> L_Y; footprint (none) -> galvanize:PinHeader_1x03_P2.54mm_Vertical_Labeled
- J17: renamed from J?; value Conn_01x03 -> R_X; footprint (none) -> galvanize:PinHeader_1x03_P2.54mm_Vertical_Labeled
- J18: renamed from J?; value Conn_01x03 -> R_Y; footprint (none) -> galvanize:PinHeader_1x03_P2.54mm_Vertical_Labeled
- J19: renamed from J?; value Conn_01x03 -> L_Tr; footprint (none) -> galvanize:PinHeader_1x03_P2.54mm_Vertical_Labeled
- J2: renamed from J?; value Conn_01x02 -> LEFT; footprint (none) -> galvanize:PinHeader_1x02_P2.54mm_Vertical_Labeled
- J20: renamed from J?; value Conn_01x03 -> R_Tr; footprint (none) -> galvanize:PinHeader_1x03_P2.54mm_Vertical_Labeled
- J3: renamed from J?; value Conn_01x02 -> DOWN; footprint (none) -> galvanize:PinHeader_1x02_P2.54mm_Vertical_Labeled
- J4: renamed from J?; value Conn_01x02 -> UP; footprint (none) -> galvanize:PinHeader_1x02_P2.54mm_Vertical_Labeled
- J5: renamed from J?; value Conn_01x02 -> B1; footprint (none) -> galvanize:PinHeader_1x02_P2.54mm_Vertical_Labeled
- J6: renamed from J?; value Conn_01x02 -> B2; footprint (none) -> galvanize:PinHeader_1x02_P2.54mm_Vertical_Labeled
- J7: renamed from J?; value Conn_01x02 -> B3; footprint (none) -> galvanize:PinHeader_1x02_P2.54mm_Vertical_Labeled
- J8: renamed from J?; value Conn_01x02 -> B4; footprint (none) -> galvanize:PinHeader_1x02_P2.54mm_Vertical_Labeled
- J9: renamed from J?; value Conn_01x02 -> B5; footprint (none) -> galvanize:PinHeader_1x02_P2.54mm_Vertical_Labeled
- U1: renamed from U?; footprint (none) -> Teensy:Teensy30_31_32_LC
Connections:
- net 3V3: now also J15.2 (Pin_2), J16.2 (Pin_2), J17.2 (Pin_2), J18.2 (Pin_2), J19.2 (Pin_2), J20.2 (Pin_2), C3.2
- net GND: now also J1.2 (Pin_2), J10.2 (Pin_2), J11.2 (Pin_2), J12.2 (Pin_2), J13.2 (Pin_2), J14.2 (Pin_2), J15.3 (Pin_3), J16.3 (Pin_3), J17.3 (Pin_3), J18.3 (Pin_3), J19.3 (Pin_3), J2.2 (Pin_2), J20.3 (Pin_3), J3.2 (Pin_2), J4.2 (Pin_2), J5.2 (Pin_2), J6.2 (Pin_2), J7.2 (Pin_2), J8.2 (Pin_2), J9.2 (Pin_2), C1.1, C2.1, C3.1
- net PIN_10: now also J13.1 (Pin_1)
- net PIN_11: now also J14.1 (Pin_1)
- net PIN_14: now also J15.1 (Pin_1)
- net PIN_15: now also J16.1 (Pin_1)
- net PIN_16: now also J17.1 (Pin_1)
- net PIN_17: now also J18.1 (Pin_1)
- net PIN_18: now also J19.1 (Pin_1)
- net PIN_19: now also J20.1 (Pin_1)
- net PIN_2: now also J5.1 (Pin_1)
- net PIN_20: now also J1.1 (Pin_1)
- net PIN_21: now also J2.1 (Pin_1)
- net PIN_22: now also J3.1 (Pin_1)
- net PIN_23: now also J4.1 (Pin_1)
- net PIN_3: now also J6.1 (Pin_1)
- net PIN_4: now also J7.1 (Pin_1)
- net PIN_5: now also J8.1 (Pin_1)
- net PIN_6: now also J9.1 (Pin_1)
- net PIN_7: now also J10.1 (Pin_1)
- net PIN_8: now also J11.1 (Pin_1)
- net PIN_9: now also J12.1 (Pin_1)
- net VIN: now also C1.2, C2.2
- net PIN_0: no longer names the net of U1.2 (0_RX1_MOSI1_Touch)
- net PIN_1: no longer names the net of U1.3 (1_TX1_MISO1_Touch)
- net PIN_12: no longer names the net of U1.14 (12_MISO0)
- net PIN_13: no longer names the net of U1.20 (13_LED_SCK0)
- no-connect marks 0 -> 15
Other:
- note added: "Galvanize: Teesnsy based USB xinput joystick board"
